File: PCB/all.brd (EAGLE design)
At the start: 45 x 45 mm, 120 parts, among them J1 ISP Programmer, J2 LIPO-BATTERY-CONNECTOR, J3 Qi coil, J4 Qi coil, J5 Qi coil, J6 Qi coil, J7 UART, J8 BL-HP20AUW2C, Q1 NPN, Q2 NPN, U1 ATTINY1634MLF20, U2 LM3671, U3 MPU-6050-1, U4 BQ51013B_RHL_20, U5 MCP73831, U6 CAT4139, U7 BQ51013B_RHL_20, U8 BQ51013B_RHL_20, U9 BQ51013B_RHL_20

Commit message: fabrication output generated
Parts:
- added FD1, FD2: FIDUCIAL1X2, SparkFun-Aesthetics:FIDUCIAL-1X2
- SJ1, SJ2: device SparkFun-Retired:SJ_3_PASTE2&3 -> SparkFun-Passives:PAD-JUMPER-3-2OF3_NC_BY_TRACE_YES_SILK_FULL_BOX
- moved SJ1 0.15 mm to (21.9, 14.9), turned to 180 degrees
- moved SJ2 0.11 mm to (23.8, 12.0), turned to 180 degrees
Connections:
- net +5V: now also SJ2.1; no longer SJ2.3
- net N$3: now also SJ1.1; no longer SJ1.3
- net N$4: now also SJ1.3; no longer SJ1.1
- net N$64: now also SJ2.3; no longer SJ2.1
Routing:
- net N$3: track 4.40 -> 5.21 mm
- net N$67: track 0.00 -> 0.81 mm

Commit message: going back to 32u4
Parts:
- removed J7: UART, SparkFun-Connectors:1X02
- removed R1: 10k, rcl:R0603
- added C2: 1µF, rcl:C0603
- added C23, C3: 18p, rcl:C0603
- added F2: PTC0603, SparkFun-PowerIC:0603
- added Q3: 8MHz, pero_library:6X3.2MM
- added R21: 10k, rcl:R0603
- added R23, R24: 22, rcl:R0603
- added S1: Reset, pero_library:TACTILE-SWITCH-SKSGAAE010
- J1: value ISP Programmer -> micro USB; device SparkFun:2X3 -> SparkFun-Connectors:USB-B-MICRO-SMD_V03
- L2: value 22uH -> 2.2uH
- U1: value ATTINY1634MLF20 -> ATMEGA32U4QFN; device attiny1634:MLF20 -> SparkFun-DigitalIC:QFN-44
- moved U1 181.9 mm to (-113.8, -86.4), turned to 0 degrees
- moved J1 167.5 mm to (-112.8, -73.2), turned to 0 degrees
Connections:
- removed net MISO: J1.1, U1.17
- removed net RX: J7.1, U1.20
- removed net TX: J7.2, U1.19
- new net N$71: C23.2, Q3.P$2, U1.17
- new net N$72: C3.2, Q3.P$1, U1.16
- new net N$73: F2.1, J1.VBUS
- new net N$74: J1.D+, R23.1
- new net N$78: J1.D-, R24.1
- new net N$80: R23.2, U1.4
- new net N$81: R24.2, U1.3
- new net VUSB: F2.2, U1.7
- net +5V: no longer J1.2
- net 3.3V: now also C2.1, R21.2, U1.14, U1.24, U1.34, U1.44, U1.6; no longer R1.2, U1.9
- net GND: now also C2.2, C23.1, C3.1, J1.GND, S1.P$1, S1.P$3, U1.15, U1.23, U1.35, U1.43, U1.5; no longer J1.6, U1.8, U1.GND
- net PWM: no longer U1.15
- net RGB: no longer U1.1
- net RST: now also R21.1, S1.P$2, S1.P$4, U1.13; no longer J1.5, R1.1, U1.12
- net SCL: now also U1.18; no longer J1.3, U1.14
- net SDA: now also U1.19; no longer J1.4, U1.18
Routing:
- net SDA: track 21.1 -> 9.71 mm
- net RST: track 7.48 -> 0.00 mm
- net MISO: track 4.80 -> 0.00 mm
- net RX: track 3.48 -> 0.00 mm
- net TX: track 3.24 -> 0.00 mm
- net 3.3V: track 51.7 -> 48.4 mm
- net +5V: track 85.5 -> 82.8 mm
- net SCL: track 22.7 -> 20.1 mm
- net GND: track 66.5 -> 64.5 mm, vias 49 -> 48
- net RGB: track 5.02 -> 3.87 mm

Commit message: started routing with 32u4
Parts:
- moved S1 216.3 mm to (61.0, 29.5)
- moved C2 212.2 mm to (57.9, 27.4), turned to 180 degrees
- moved R21 210.7 mm to (61.0, 27.6), turned to 180 degrees
- moved F2 206.8 mm to (46.7, 21.1), turned to 180 degrees
- moved R23 193.2 mm to (46.7, 23.7)
- moved J1 191.0 mm to (52.2, 23.1), turned to 180 degrees
- moved R24 188.6 mm to (46.7, 22.4)
- moved C3 186.7 mm to (28.1, 16.4), turned to 90 degrees
- moved U1 180.0 mm to (29.2, 23.0), turned to 270 degrees
- moved C23 172.5 mm to (35.5, 17.9), turned to 270 degrees
- moved Q3 160.0 mm to (22.8, 22.2), turned to 270 degrees
- moved JP2 25.8 mm to (62.8, 17.6)
- moved R5 25.8 mm to (61.1, 15.3)
- moved C14 25.8 mm to (60.1, 20.8)
- moved C7 13.4 mm to (27.0, 16.4), turned to 270 degrees
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Routing:
- net +5V: track 82.8 -> 68.2 mm
- net 3.3V: track 48.4 -> 57.0 mm
- net SCL: track 20.1 -> 13.1 mm
- net PWM: track 12.3 -> 5.80 mm, vias 1 -> 0
- net N$71: track 0.00 -> 4.96 mm
- net N$72: track 0.00 -> 3.36 mm
- net N$64: track 8.20 -> 8.91 mm
- net GND: vias 48 -> 46
Other:
- board text removed: "MISO"
- board text removed: "Rx"
- board text removed: "Tx"

Commit message: routing finished
Parts:
- added C4: 0.1μF, rcl:C0603K
- CP1, CP3, CP5, CP7: value 18pF -> 2.2nF
- CP2, CP4, CP6, CP8, CS, CS10, CS27, CS30: value 18pF -> x
- CS17, CS20, CS37, CS7: value 18pF -> 220nF
- moved R5 31.3 mm to (29.8, 17.5), turned to 90 degrees
- moved JP2 30.8 mm to (32.0, 17.3), turned to 0 degrees
- moved R21 29.6 mm to (31.5, 26.7), turned to 0 degrees
- moved S1 27.9 mm to (33.6, 24.1), turned to 270 degrees
- moved C2 26.7 mm to (31.5, 23.1), turned to 270 degrees
- moved C14 25.1 mm to (35.0, 19.9), turned to 180 degrees
- moved C23 19.0 mm to (20.4, 29.4), turned to 90 degrees
- moved C3 13.8 mm to (28.4, 30.2)
- moved C6 11.8 mm to (23.1, 18.6), turned to 180 degrees
- moved C9 11.0 mm to (27.6, 18.4), turned to 180 degrees
- moved C7 9.94 mm to (20.8, 24.2)
- moved R24 9.71 mm to (37.1, 23.4), turned to 180 degrees
- moved R23 9.67 mm to (37.1, 24.9), turned to 180 degrees
- moved F2 9.67 mm to (37.1, 21.8)
- moved J1 9.14 mm to (43.0, 23.1)
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Connections:
- net 3.3V: now also C4.1
- net GND: now also C4.2
- net PWM: now also U1.12
- net RGB: now also U1.1
Routing:
- net 3.3V: track 57.0 -> 97.5 mm, vias 0 -> 4
- net GND: track 64.5 -> 94.1 mm, vias 46 -> 47
- net PWM: track 5.80 -> 19.7 mm, vias 0 -> 1
- net VUSB: track 0.00 -> 12.3 mm, vias 0 -> 2
- net +5V: track 68.2 -> 80.4 mm, vias 3 -> 4
- net N$81: track 0.00 -> 8.82 mm
- net N$80: track 0.00 -> 8.06 mm
- net RST: track 0.00 -> 7.44 mm
- net N$71: track 4.96 -> 8.90 mm
- net N$74: track 0.00 -> 3.74 mm
- net N$62: track 3.55 -> 6.64 mm
- net N$78: track 0.00 -> 2.77 mm
- net N$72: track 3.36 -> 5.98 mm
- net V_QI_IN: track 84.2 -> 86.8 mm
- net N$73: track 0.00 -> 2.41 mm
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Other:
- board text added: "+"
- board text added: "Board layout 14.11.2016"
- board text added: "Loveread Lamp v3.0 Pero 2016"
- board text added: "Nov. 2016"
- board text added: "RGB"
- board text added: "v3.0"
- board text removed: "Board layout 26.7.2016"
- board text removed: "July, 2016"
- board text removed: "Loveread Lamp v2.0 Pero 2016"
- board text removed: "MOSI"
- board text removed: "v2.0"

Commit message: order complete
Parts:
- moved C18 0.25 mm to (3.65, 13.5)
